Commit message: update doosan driver for gachon univ

File: dsr_description/xacro/macro.m0609.white.xacro (robot description, xacro)
@@ -13,4 +13,9 @@
 					iyz="-0.00029038"
 					izz="0.020054"/>
+				<collision>
+						<geometry>
+								<cylinder radius="0.08" length="0.01"/>
+						</geometry>
+				</collision>
 			</inertial>
 			<visual>
@@ -206,4 +211,25 @@
 			</visual>
 		</link>
+		<!-- joint gripper -->
+		<joint name="joint_gripper" type="fixed">
+			<parent link="link6" />
+			<child link="link_gripper" />
+			<origin xyz="0 0 0.28" rpy="0 0 0" />  <!-- gripper length: 0.28m -->
+			<axis xyz="0 0 0" />
+		</joint>
+		<link name="link_gripper">
+			<inertial>
+				<mass value="0.3"/>
+				<origin xyz="0 0 0"/>
+				<inertia ixx="0.001" ixy="0" ixz="0" iyy="0.001" iyz="0" izz="0.001"/>
+			</inertial>
+			<visual>
+				<origin xyz="0 0 0" rpy="0 0 0" />
+				<geometry>
+					<mesh filename="package://dsr_description/meshes/gripper/plaif/gripper.dae" scale="0.001 0.001 0.001"/>
+				</geometry>
+				<color rgba="1.0 1.0 1.0 0.8"/>
+			</visual>
+		</link>
     <xacro:dsr_transmission />
     <xacro:dsr_gazebo namespace="${namespace}" />

Commit message: update joint limits

File: dsr_description/xacro/macro.m0609.white.xacro (robot description, xacro)
@@ -32,5 +32,5 @@
 			<origin rpy="0 0 0" xyz="0 0 0.1" />
 			<axis xyz="0 0 1" />
-			<limit effort="163" lower="-6.2832" upper="6.2832" velocity="2.618"/>
+			<limit effort="163" lower="0.5236" upper="2.618" velocity="2.618"/>
 			<dynamics friction="0" />
 		</joint>
@@ -61,5 +61,5 @@
 			<origin rpy="0 -1.571 -1.571" xyz="0 0.0062 0" />
 			<axis xyz="0 0 1" />
-			<limit effort="163" lower="-6.2832" upper="6.2832" velocity="2.618"/>
+			<limit effort="163" lower="-0.6981317" upper="1.0472" velocity="2.618"/>
 			<dynamics friction="0" />
 		</joint>
@@ -103,5 +103,5 @@
 			<origin rpy="0 0 1.571" xyz="0.411 0 0" />
 			<axis xyz="0 0 1" />
-			<limit effort="96" lower="-2.618" upper="2.618" velocity="3.1416"/>
+			<limit effort="96" lower="0.5236" upper="2.618" velocity="3.1416"/>
 			<dynamics friction="0" />
 		</joint>
@@ -127,5 +127,5 @@
 			<origin rpy="1.571 0 0" xyz="0 -0.368 0" />
 			<axis xyz="0 0 1" />
-			<limit effort="50" lower="-6.2832" upper="6.2832" velocity="3.927"/>
+			<limit effort="50" lower="-0.6981317" upper="0.6981317" velocity="3.927"/>
 			<dynamics friction="0" />
 		</joint>
@@ -163,5 +163,5 @@
 			<origin rpy="-1.571 0 0" xyz="0 0 0" />
 			<axis xyz="0 0 1" />
-			<limit effort="50" lower="-6.2832" upper="6.2832" velocity="3.927"/>
+			<limit effort="50" lower="0.8726646" upper="2.268928" velocity="3.927"/>
 			<dynamics friction="0" />
 		</joint>
@@ -193,5 +193,5 @@
 			<origin rpy="1.571 0 0" xyz="0 -0.121 0" />
 			<axis xyz="0 0 1" />
-			<limit effort="50" lower="-6.2832" upper="6.2832" velocity="3.927"/>
+			<limit effort="50" lower="-3.12414" upper="3.12414" velocity="3.927"/>
 			<dynamics friction="0" />
 		</joint>

Commit message: update link names

File: dsr_description/xacro/macro.m0609.white.xacro (robot description, xacro)
@@ -6,5 +6,5 @@
 	<xacro:macro name="m0609" params="namespace">
     <xacro:dsr_materials />
-		<link name="base_0">
+		<link name="base_link">
 			<inertial>
 				<mass value="3.18"/>
@@ -28,5 +28,5 @@
 		<!-- joint 1 -->
 		<joint name="joint1" type="revolute">
-			<parent link="base_0" />
+			<parent link="base_link" />
 			<child link="link1" />
 			<origin rpy="0 0 0" xyz="0 0 0.1" />
@@ -211,25 +211,33 @@
 			</visual>
 		</link>
-		<!-- joint gripper -->
+		<!-- tool0 -->
+		<link name="tool0" />
+		<joint name="joint_tool0" type="fixed">
+			<parent link="link6" />
+			<child link="tool0" />
+			<origin xyz="0 0 0" rpy="0 0 -1.57" />
+			<axis xyz="0 0 0" />
+		</joint>
+		<!-- gripper -->
+		<link name="link_gripper">
+			<inertial>
+				<mass value="0.3"/>
+				<origin xyz="0 0 0"/>
+				<inertia ixx="0.001" ixy="0" ixz="0" iyy="0.001" iyz="0" izz="0.001"/>
+			</inertial>
+			<visual>
+				<origin xyz="0 0 0" rpy="0 0 0" />
+				<geometry>
+					<mesh filename="package://dsr_description/meshes/gripper/plaif/gripper.dae" scale="0.001 0.001 0.001"/>
+				</geometry>
+				<color rgba="1.0 1.0 1.0 0.8"/>
+			</visual>
+		</link>
 		<joint name="joint_gripper" type="fixed">
-			<parent link="link6" />
+			<parent link="tool0" />
 			<child link="link_gripper" />
 			<origin xyz="0 0 0.28" rpy="0 0 0" />  <!-- gripper length: 0.28m -->
 			<axis xyz="0 0 0" />
 		</joint>
-		<link name="link_gripper">
-			<inertial>
-				<mass value="0.3"/>
-				<origin xyz="0 0 0"/>
-				<inertia ixx="0.001" ixy="0" ixz="0" iyy="0.001" iyz="0" izz="0.001"/>
-			</inertial>
-			<visual>
-				<origin xyz="0 0 0" rpy="0 0 0" />
-				<geometry>
-					<mesh filename="package://dsr_description/meshes/gripper/plaif/gripper.dae" scale="0.001 0.001 0.001"/>
-				</geometry>
-				<color rgba="1.0 1.0 1.0 0.8"/>
-			</visual>
-		</link>
     <xacro:dsr_transmission />
     <xacro:dsr_gazebo namespace="${namespace}" />
